File: 1s_lipo.kicad_sch (KiCad schematic)
At the start: 23 parts, among them J3 LiPo 1S, U6 DW01, U7 TLV62569DBV, U8 PM8205A, U9 HX4054A

Commit message: Changed FETs to SOT-23 and buttons to something that is more boring
Parts:
- C10: LCSC (none) -> C1634
- C11, C8: LCSC (none) -> C14663
- C12: LCSC (none) -> C19666
- C13, C14, C9: LCSC (none) -> C19702
- D514: LCSC (none) -> C72041
- J3, L1, U7, U8, U9: LCSC (none) -> DNP
- R10: LCSC (none) -> C22775
- R11, R15: LCSC (none) -> C21190
- R12, R13, R14: LCSC (none) -> C22936
- R16: LCSC (none) -> C22975
- R17: LCSC (none) -> C23146
- R18: LCSC (none) -> C23254
Changed lines of the file:
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@@
+      (effects (font (size 1.27 1.27)) hide)
+    )
+    (property "LCSC" "DNP" (id 4) (at 223.52 91.44 0)
       (effects (font (size 1.27 1.27)) hide)
     )
@@
       (effects (font (size 1.27 1.27)) hide)
     )
+    (property "LCSC" "C22775" (id 4) (at 57.15 50.8 0)
+      (effects (font (size 1.27 1.27)) hide)
+    )
   )
   (symbol (lib_id "Device:R") (at 58.42 137.16 180) (unit 1)
@@
       (effects (font (size 1.27 1.27)) hide)
     )
+    (property "LCSC" "C22936" (id 4) (at 58.42 137.16 0)
+      (effects (font (size 1.27 1.27)) hide)
+    )
   )
   (symbol (lib_id "Device:R") (at 71.12 137.16 180) (unit 1)
@@
       (effects (font (size 1.27 1.27)) hide)
     )
+    (property "LCSC" "C21190" (id 4) (at 71.12 137.16 0)
+      (effects (font (size 1.27 1.27)) hide)
+    )
   )
   (symbol (lib_id "Device:R") (at 83.82 125.73 180) (unit 1)
@@
       (effects (font (size 1.27 1.27)) hide)
     )
+    (property "LCSC" "C22936" (id 4) (at 83.82 125.73 0)
+      (effects (font (size 1.27 1.27)) hide)
+    )
   )
   (symbol (lib_id "Device:R") (at 95.25 125.73 180) (unit 1)
@@
       (effects (font (size 1.27 1.27)) hide)
     )
+    (property "LCSC" "C22936" (id 4) (at 95.25 125.73 0)
+      (effects (font (size 1.27 1.27)) hide)
+    )
   )
   (symbol (lib_id "Device:R") (at 106.68 161.29 180) (unit 1)
@@
       (effects (font (size 1.27 1.27)) hide)
     )
+    (property "LCSC" "C22975" (id 4) (at 106.68 161.29 0)
+      (effects (font (size 1.27 1.27)) hide)
+    )
   )
   (symbol (lib_id "Device:R") (at 113.03 68.58 180) (unit 1)
@@
       (effects (font (size 1.27 1.27)) hide)
     )
+    (property "LCSC" "C21190" (id 4) (at 113.03 68.58 0)
+      (effects (font (size 1.27 1.27)) hide)
+    )
   )
   (symbol (lib_id "Device:R") (at 228.6 97.79 180) (unit 1)
@@
       (effects (font (size 1.27 1.27)) hide)
     )
+    (property "LCSC" "C23146" (id 4) (at 228.6 97.79 0)
+      (effects (font (size 1.27 1.27)) hide)
+    )
   )
   (symbol (lib_id "Device:R") (at 228.6 107.95 0) (unit 1)
@@
     )
     (property "PN_1" "0201WMF8202TCE" (id 7) (at 228.6 107.95 0)
+      (effects (font (size 1.27 1.27)) hide)
+    )
+    (property "LCSC" "C23254" (id 4) (at 228.6 107.95 0)
       (effects (font (size 1.27 1.27)) hide)
     )
@@
       (effects (font (size 1.27 1.27)) hide)
     )
+    (property "LCSC" "DNP" (id 4) (at 39.37 50.8 0)
+      (effects (font (size 1.27 1.27)) hide)
+    )
   )
   (symbol (lib_id "Device:LED_ALT") (at 71.12 148.59 90) (unit 1)
@@
       (effects (font (size 1.27 1.27)) hide)
     )
+    (property "LCSC" "C72041" (id 4) (at 71.12 148.59 0)
+      (effects (font (size 1.27 1.27)) hide)
+    )
   )
   (symbol (lib_id "Device:C") (at 58.42 148.59 0) (unit 1)
@@
       (effects (font (size 1.27 1.27)) hide)
     )
+    (property "LCSC" "C14663" (id 4) (at 58.42 148.59 0)
+      (effects (font (size 1.27 1.27)) hide)
+    )
   )
   (symbol (lib_id "Device:C") (at 66.04 55.88 0) (unit 1)
@@
       (effects (font (size 1.27 1.27)) hide)
     )
+    (property "LCSC" "C14663" (id 4) (at 66.04 55.88 0)
+      (effects (font (size 1.27 1.27)) hide)
+    )
   )
   (symbol (lib_id "Device:C") (at 111.76 153.67 0) (unit 1)
@@
       (effects (font (size 1.27 1.27)) hide)
     )
+    (property "LCSC" "C19666" (id 4) (at 111.76 153.67 0)
+      (effects (font (size 1.27 1.27)) hide)
+    )
   )
   (symbol (lib_id "Device:C") (at 185.42 96.52 0) (mirror x) (unit 1)
@@
       (effects (font (size 1.27 1.27)) hide)
     )
+    (property "LCSC" "C19702" (id 4) (at 185.42 96.52 0)
+      (effects (font (size 1.27 1.27)) hide)
+    )
   )
   (symbol (lib_id "Device:C") (at 233.68 97.79 180) (unit 1)
@@
       (effects (font (size 1.27 1.27)) hide)
     )
+    (property "LCSC" "C1634" (id 4) (at 233.68 97.79 0)
+      (effects (font (size 1.27 1.27)) hide)
+    )
   )
   (symbol (lib_id "Device:C") (at 247.65 96.52 0) (mirror x) (unit 1)
@@
       (effects (font (size 1.27 1.27)) hide)
     )
+    (property "LCSC" "C19702" (id 4) (at 247.65 96.52 0)
+      (effects (font (size 1.27 1.27)) hide)
+    )
   )
   (symbol (lib_id "Device:C") (at 252.73 96.52 180) (unit 1)
@@
     )
     (property "PN_1" "CC0402MRX5R5BB106" (id 7) (at 252.73 96.52 0)
+      (effects (font (size 1.27 1.27)) hide)
+    )
+    (property "LCSC" "C19702" (id 4) (at 252.73 96.52 0)
       (effects (font (size 1.27 1.27)) hide)
     )
@@
       (effects (font (size 1.27 1.27)) hide)
     )
+    (property "LCSC" "DNP" (id 4) (at 208.28 102.87 0)
+      (effects (font (size 1.27 1.27)) hide)
+    )
   )
   (symbol (lib_id "pm8205a:PM8205A") (at 91.44 77.47 0) (unit 1)
@@
       (effects (font (size 1.27 1.27)) hide)
     )
+    (property "LCSC" "DNP" (id 4) (at 91.44 77.47 0)
+      (effects (font (size 1.27 1.27)) hide)
+    )
   )
   (symbol (lib_id "hx4054a:HX4054A") (at 90.17 151.13 0) (unit 1)
@@
       (effects (font (size 1.27 1.27)) hide)
     )
+    (property "LCSC" "DNP" (id 4) (at 90.17 151.13 0)
+      (effects (font (size 1.27 1.27)) hide)
+    )
