File: badge.kicad_sch (KiCad schematic)
At the start: 7 parts, among them SW1 A, SW2 B, SW3 X, SW4 Y, X1 #badgelife

Commit message: Changed FETs to SOT-23 and buttons to something that is more boring
Parts:
- SW1, SW2, SW3, SW4: footprint Buttons:SW_SPST_TS3625A-HT -> tom-mechanical:SW_SPST_SMD_2PIN_3.5x6.0; LCSC (none) -> DNP
- X1: LCSC (none) -> DNP
Changed lines of the file:
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@@
     (property "Reference" "SW1" (id 0) (at 151.13 133.35 0))
     (property "Value" "A" (id 1) (at 151.13 135.89 0))
-    (property "Footprint" "Buttons:SW_SPST_TS3625A-HT" (id 2) (at 151.13 139.7 0)
+    (property "Footprint" "tom-mechanical:SW_SPST_SMD_2PIN_3.5x6.0" (id 2) (at 151.13 139.7 0)
       (effects (font (size 1.27 1.27)) hide)
     )
     (property "Datasheet" "~" (id 3) (at 151.13 139.7 0)
+      (effects (font (size 1.27 1.27)) hide)
+    )
+    (property "LCSC" "DNP" (id 4) (at 151.13 139.7 0)
       (effects (font (size 1.27 1.27)) hide)
     )
@@
     (property "Reference" "SW2" (id 0) (at 151.13 143.51 0))
     (property "Value" "B" (id 1) (at 151.13 146.05 0))
-    (property "Footprint" "Buttons:SW_SPST_TS3625A-HT" (id 2) (at 151.13 149.86 0)
+    (property "Footprint" "tom-mechanical:SW_SPST_SMD_2PIN_3.5x6.0" (id 2) (at 151.13 149.86 0)
       (effects (font (size 1.27 1.27)) hide)
     )
     (property "Datasheet" "~" (id 3) (at 151.13 149.86 0)
+      (effects (font (size 1.27 1.27)) hide)
+    )
+    (property "LCSC" "DNP" (id 4) (at 151.13 149.86 0)
       (effects (font (size 1.27 1.27)) hide)
     )
@@
     (property "Reference" "SW3" (id 0) (at 151.13 153.67 0))
     (property "Value" "X" (id 1) (at 151.13 156.21 0))
-    (property "Footprint" "Buttons:SW_SPST_TS3625A-HT" (id 2) (at 151.13 160.02 0)
+    (property "Footprint" "tom-mechanical:SW_SPST_SMD_2PIN_3.5x6.0" (id 2) (at 151.13 160.02 0)
       (effects (font (size 1.27 1.27)) hide)
     )
     (property "Datasheet" "~" (id 3) (at 151.13 160.02 0)
+      (effects (font (size 1.27 1.27)) hide)
+    )
+    (property "LCSC" "DNP" (id 4) (at 151.13 160.02 0)
       (effects (font (size 1.27 1.27)) hide)
     )
@@
     (property "Reference" "SW4" (id 0) (at 151.13 163.83 0))
     (property "Value" "Y" (id 1) (at 151.13 166.37 0))
-    (property "Footprint" "Buttons:SW_SPST_TS3625A-HT" (id 2) (at 151.13 170.18 0)
+    (property "Footprint" "tom-mechanical:SW_SPST_SMD_2PIN_3.5x6.0" (id 2) (at 151.13 170.18 0)
       (effects (font (size 1.27 1.27)) hide)
     )
     (property "Datasheet" "~" (id 3) (at 151.13 170.18 0)
+      (effects (font (size 1.27 1.27)) hide)
+    )
+    (property "LCSC" "DNP" (id 4) (at 151.13 170.18 0)
       (effects (font (size 1.27 1.27)) hide)
     )
@@
       (effects (font (size 1.27 1.27)) hide)
     )
+    (property "LCSC" "DNP" (id 4) (at 222.25 95.25 0)
+      (effects (font (size 1.27 1.27)) hide)
+    )
   )
   (sheet (at 198.12 118.11) (size 48.26 27.94)
@@
     )
     (path "/e88db032-369f-4dcc-9e5f-89425dc60d66"
-      (reference "SW1") (unit 1) (value "A") (footprint "Buttons:SW_SPST_TS3625A-HT")
+      (reference "SW1") (unit 1) (value "A") (footprint "tom-mechanical:SW_SPST_SMD_2PIN_3.5x6.0")
     )
     (path "/cfa1c6cd-833b-4188-aa12-c63c86619375"
-      (reference "SW2") (unit 1) (value "B") (footprint "Buttons:SW_SPST_TS3625A-HT")
+      (reference "SW2") (unit 1) (value "B") (footprint "tom-mechanical:SW_SPST_SMD_2PIN_3.5x6.0")
     )
     (path "/ef61248f-b66a-497b-ab52-4440eebad450"
-      (reference "SW3") (unit 1) (value "X") (footprint "Buttons:SW_SPST_TS3625A-HT")
+      (reference "SW3") (unit 1) (value "X") (footprint "tom-mechanical:SW_SPST_SMD_2PIN_3.5x6.0")
     )
     (path "/a8418c84-7faf-4f0a-9262-5bb08949bdc3"
-      (reference "SW4") (unit 1) (value "Y") (footprint "Buttons:SW_SPST_TS3625A-HT")
+      (reference "SW4") (unit 1) (value "Y") (footprint "tom-mechanical:SW_SPST_SMD_2PIN_3.5x6.0")
     )
     (path "/257d8dda-dcb6-4e08-9333-cf5bc17f4872"
@@
     )
     (path "/9d1ab8a7-551e-4acd-bdbd-902f3132e84e/00000000-0000-0000-0000-00005eeea025"
-      (reference "R9") (unit 1) (value "4.7K") (footprint "Resistor_SMD:R_0603_1608Metric")
+      (reference "R9") (unit 1) (value "4.7k") (footprint "Resistor_SMD:R_0603_1608Metric")
     )
     (path "/9d1ab8a7-551e-4acd-bdbd-902f3132e84e/00000000-0000-0000-0000-00005ed13ce9"
@@
     )
     (path "/82f21894-a473-468f-9e64-7bc4d6d80b53/ef1d04ac-171a-493f-b4b5-1daf45840274"
-      (reference "Q1") (unit 1) (value "3412") (footprint "Package_TO_SOT_SMD:SOT-883")
+      (reference "Q1") (unit 1) (value "3412") (footprint "Package_TO_SOT_SMD:SOT-23")
     )
     (path "/82f21894-a473-468f-9e64-7bc4d6d80b53/4776a220-6975-44aa-9000-2ed95a476041"
-      (reference "Q2") (unit 1) (value "3412") (footprint "Package_TO_SOT_SMD:SOT-883")
+      (reference "Q2") (unit 1) (value "3412") (footprint "Package_TO_SOT_SMD:SOT-23")
     )
     (path "/82f21894-a473-468f-9e64-7bc4d6d80b53/7f68c60f-4f92-4e7c-9b0c-73f77b1bc050"
-      (reference "Q3") (unit 1) (value "3412") (footprint "Package_TO_SOT_SMD:SOT-883")
+      (reference "Q3") (unit 1) (value "3412") (footprint "Package_TO_SOT_SMD:SOT-23")
     )
     (path "/82f21894-a473-468f-9e64-7bc4d6d80b53/245354e6-bc31-425a-b709-8ac471a35478"
-      (reference "Q4") (unit 1) (value "3412") (footprint "Package_TO_SOT_SMD:SOT-883")
+      (reference "Q4") (unit 1) (value "3412") (footprint "Package_TO_SOT_SMD:SOT-23")
     )
     (path "/82f21894-a473-468f-9e64-7bc4d6d80b53/204df76e-fb1d-4a82-a22f-52f847de26ed"
-      (reference "Q5") (unit 1) (value "3412") (footprint "Package_TO_SOT_SMD:SOT-883")
+      (reference "Q5") (unit 1) (value "3412") (footprint "Package_TO_SOT_SMD:SOT-23")
     )
     (path "/82f21894-a473-468f-9e64-7bc4d6d80b53/05128dc3-3c75-4fbc-83d1-6e936f7b666d"
-      (reference "Q6") (unit 1) (value "3412") (footprint "Package_TO_SOT_SMD:SOT-883")
+      (reference "Q6") (unit 1) (value "3412") (footprint "Package_TO_SOT_SMD:SOT-23")
     )
     (path "/82f21894-a473-468f-9e64-7bc4d6d80b53/b3677eac-f98d-456f-a21e-b0420b033a6d"
-      (reference "Q7") (unit 1) (value "3412") (footprint "Package_TO_SOT_SMD:SOT-883")
+      (reference "Q7") (unit 1) (value "3412") (footprint "Package_TO_SOT_SMD:SOT-23")
     )
     (path "/82f21894-a473-468f-9e64-7bc4d6d80b53/1aa33725-4f1f-46fc-ab09-95c8fe2a63ec"
-      (reference "Q8") (unit 1) (value "3412") (footprint "Package_TO_SOT_SMD:SOT-883")
+      (reference "Q8") (unit 1) (value "3412") (footprint "Package_TO_SOT_SMD:SOT-23")
     )
     (path "/82f21894-a473-468f-9e64-7bc4d6d80b53/762906a3-a060-40c3-8ec6-79853fb53d6d"
-      (reference "Q9") (unit 1) (value "3412") (footprint "Package_TO_SOT_SMD:SOT-883")
+      (reference "Q9") (unit 1) (value "3412") (footprint "Package_TO_SOT_SMD:SOT-23")
     )
     (path "/82f21894-a473-468f-9e64-7bc4d6d80b53/8f419ad8-fb0d-4990-8917-15e8bd7b610a"
-      (reference "Q10") (unit 1) (value "3412") (footprint "Package_TO_SOT_SMD:SOT-883")
+      (reference "Q10") (unit 1) (value "3412") (footprint "Package_TO_SOT_SMD:SOT-23")
     )
     (path "/82f21894-a473-468f-9e64-7bc4d6d80b53/7c8f5cc2-e7a0-4691-bd2c-029e5fbbf477"
-      (reference "Q11") (unit 1) (value "3412") (footprint "Package_TO_SOT_SMD:SOT-883")
+      (reference "Q11") (unit 1) (value "3412") (footprint "Package_TO_SOT_SMD:SOT-23")
     )
     (path "/82f21894-a473-468f-9e64-7bc4d6d80b53/d60f1bd8-132f-47c6-9a0a-79b611ecac9a"
-      (reference "Q12") (unit 1) (value "3412") (footprint "Package_TO_SOT_SMD:SOT-883")
+      (reference "Q12") (unit 1) (value "3412") (footprint "Package_TO_SOT_SMD:SOT-23")
     )
     (path "/82f21894-a473-468f-9e64-7bc4d6d80b53/e11e1f16-cc59-4e5e-bfba-9db7a5ac7d31"
-      (reference "Q13") (unit 1) (value "3412") (footprint "Package_TO_SOT_SMD:SOT-883")
+      (reference "Q13") (unit 1) (value "3412") (footprint "Package_TO_SOT_SMD:SOT-23")
     )
     (path "/82f21894-a473-468f-9e64-7bc4d6d80b53/3d482f4c-98ce-42c2-ab80-d3f0e2f52339"
-      (reference "Q14") (unit 1) (value "3412") (footprint "Package_TO_SOT_SMD:SOT-883")
+      (reference "Q14") (unit 1) (value "3412") (footprint "Package_TO_SOT_SMD:SOT-23")
     )
     (path "/82f21894-a473-468f-9e64-7bc4d6d80b53/c171bef7-b024-46a5-b831-a5672f0434d6"
-      (reference "Q15") (unit 1) (value "3412") (footprint "Package_TO_SOT_SMD:SOT-883")
+      (reference "Q15") (unit 1) (value "3412") (footprint "Package_TO_SOT_SMD:SOT-23")
     )
     (path "/82f21894-a473-468f-9e64-7bc4d6d80b53/c0abdafa-b900-420a-9d64-860358e29cc2"
-      (reference "Q16") (unit 1) (value "3412") (footprint "Package_TO_SOT_SMD:SOT-883")
+      (reference "Q16") (unit 1) (value "3412") (footprint "Package_TO_SOT_SMD:SOT-23")
     )
     (path "/82f21894-a473-468f-9e64-7bc4d6d80b53/bca6514e-a885-4f60-8ad0-b3e6c5d1f873"
