File: ledStripe.kicad_sch (KiCad schematic)
At the start: 32 parts

Commit message: Changed FETs to SOT-23 and buttons to something that is more boring
Parts:
- D1: renamed from D481; LCSC (none) -> C397045
- D10: renamed from D490; LCSC (none) -> C397045
- D11: renamed from D491; LCSC (none) -> C397045
- D12: renamed from D492; LCSC (none) -> C397045
- D13: renamed from D493; LCSC (none) -> C397045
- D14: renamed from D494; LCSC (none) -> C397045
- D15: renamed from D495; LCSC (none) -> C397045
- D16: renamed from D496; LCSC (none) -> C397045
- D17: renamed from D497; LCSC (none) -> C397045
- D18: renamed from D498; LCSC (none) -> C397045
- D19: renamed from D499; LCSC (none) -> C397045
- D2: renamed from D482; LCSC (none) -> C397045
- D20: renamed from D500; LCSC (none) -> C397045
- D21: renamed from D501; LCSC (none) -> C397045
- D22: renamed from D502; LCSC (none) -> C397045
- D23: renamed from D503; LCSC (none) -> C397045
- D24: renamed from D504; LCSC (none) -> C397045
- D25: renamed from D505; LCSC (none) -> C397045
- D26: renamed from D506; LCSC (none) -> C397045
- D27: renamed from D507; LCSC (none) -> C397045
- D28: renamed from D508; LCSC (none) -> C397045
- D29: renamed from D509; LCSC (none) -> C397045
- D3: renamed from D483; LCSC (none) -> C397045
- D30: renamed from D510; LCSC (none) -> C397045
- D31: renamed from D511; LCSC (none) -> C397045
- D32: renamed from D512; LCSC (none) -> C397045
- D4: renamed from D484; LCSC (none) -> C397045
- D5: renamed from D485; LCSC (none) -> C397045
- D6: renamed from D486; LCSC (none) -> C397045
- D7: renamed from D487; LCSC (none) -> C397045
- D8: renamed from D488; LCSC (none) -> C397045
- D9: renamed from D489; LCSC (none) -> C397045
